File: PCBV1/UART.sch (KiCad schematic (older format))
At the start: 0 parts

Commit message: Merge of recent changes to default master (#2)
* Made a bunch of very small changes.

* Added UART, modifications to video etc.

* Minor adjustments with video connections.

* Finished video signals, added HDMI and SD connectors.
Other:
- note added: "PLACE UART TO USB IC\n\nEXAMPLES:\nCP2102N\nMCP2200-I"
Changed lines of the file:
@@
 $Descr A4 11693 8268
 encoding utf-8
-Sheet 5 8
-Title "Smart Mirror"
-Date "2021-01-21"
-Rev "1.0"
-Comp "University of Southern Denmark"
-Comment1 "SRM"
+Sheet 9 8
+Title ""
+Date ""
+Rev ""
+Comp ""
+Comment1 ""
 Comment2 ""
 Comment3 ""
 Comment4 ""
 $EndDescr
+Text Notes 4850 3850 0    50   ~ 0
+PLACE UART TO USB IC\n\nEXAMPLES:\nCP2102N\nMCP2200-I
 $EndSCHEMATC
