File: PCBV1/UART.sch (KiCad schematic (older format))
At the start: 0 parts

Commit message: Added UART, modifications to video etc.
Other:
- note added: "PLACE UART TO USB IC\n\nEXAMPLES:\nCP2102N\nMCP2200-I"
Changed lines of the file:
@@
 $Descr A4 11693 8268
 encoding utf-8
-Sheet 6 9
-Title "Smart Mirror"
-Date "2021-01-21"
-Rev "1.0"
-Comp "University of Southern Denmark"
-Comment1 "SRM"
+Sheet 9 9
+Title ""
+Date ""
+Rev ""
+Comp ""
+Comment1 ""
 Comment2 ""
 Comment3 ""
 Comment4 ""
 $EndDescr
+Text Notes 4850 3850 0    50   ~ 0
+PLACE UART TO USB IC\n\nEXAMPLES:\nCP2102N\nMCP2200-I
 $EndSCHEMATC

Commit message: Added SD filter and USB-to-UART IC.
Parts:
- added C? (x2): 4.7u, symbol Device:C
- added C? (x2): 100n, symbol Device:C
- added D? (x3): LED, symbol Device:LED
- added R?: 1k, symbol Device:R
- added R? (x3): R, symbol Device:R
- added R?: 10k, symbol Device:R
- added U?: CP2102N-A01-GQFN28, Package_DFN_QFN:QFN-28-1EP_5x5mm_P0.5mm_EP3.35x3.35mm, symbol Interface_USB:CP2102N-A01-GQFN28
Connections:
- net labels added: +3V3_USB, +5V, CTS, DATA+, DATA-, GND, RTS, RX, TX
- wire segments 0 -> 38
- no-connect marks 0 -> 13
Other:
- note added: "TO-DO: Find LEDs (+ color) and resistor value"
- note removed: "PLACE UART TO USB IC\n\nEXAMPLES:\nCP2102N\nMCP2200-I"

Commit message: Many minor changes to component footprints and schematics.
Parts:
- removed D? (x3): LED, symbol Device:LED
- added D4: 150060SS55040, Personal_Passives:150060SS55040, symbol Personal_Passives:150060SS55040
- added D5: 150060VS55040, Personal_Passives:150060SS55040, symbol Personal_Passives:150060VS55040
- added D6: 150060YS55040, Personal_Passives:150060SS55040, symbol Personal_Passives:150060YS55040
- C84, C85: renamed from C?; footprint (none) -> Capacitor_SMD:C_0603_1608Metric
- R20, R21: renamed from R?; footprint (none) -> Resistor_SMD:R_0603_1608Metric
- R22, R23, R24: renamed from R?; value R -> 180; footprint (none) -> Resistor_SMD:R_0603_1608Metric
- gave numbers to parts that had none: 3
Connections:
- net labels added: +5V_USB
- net labels removed: +5V
- wire segments 38 -> 46
Other:
- note removed: "TO-DO: Find LEDs (+ color) and resistor value"
- moved on the sheet: R23, R24

Commit message: Added NAND flash with connections, updated IO config.
Parts:
- C82, C83: footprint (none) -> Capacitor_SMD:C_0603_1608Metric
Changed lines of the file:
@@
 F 0 "C83" V 5400 2350 50  0000 C CNN
 F 1 "4.7u" V 5300 2400 50  0000 C CNN
-F 2 "" H 5388 2100 50  0001 C CNN
+F 2 "Capacitor_SMD:C_0603_1608Metric" H 5388 2100 50  0001 C CNN
 F 3 "~" H 5350 2250 50  0001 C CNN
 	1    5350 2250
@@
 F 0 "C82" V 5000 2100 50  0000 C CNN
 F 1 "4.7u" V 4900 2100 50  0000 C CNN
-F 2 "" H 4988 2100 50  0001 C CNN
+F 2 "Capacitor_SMD:C_0603_1608Metric" H 4988 2100 50  0001 C CNN
 F 3 "~" H 4950 2250 50  0001 C CNN
 	1    4950 2250

Commit message: Laid final hands on Wi-Fi and all circuits. Started work on PCB.
Parts:
- renumbered C82 to C111, C83 to C112, C84 to C113, C85 to C114, R20 to R37, R21 to R38, R22 to R39, R23 to R40, R24 to R41, U9 to U13
Changed lines of the file:
@@
 Sheet 8 8
 Title "Smart Mirror"
-Date "2022-04-22"
+Date "2022-05-11"
 Rev "1.0"
 Comp "University of Southern Denmark"
@@
 $EndDescr
 $Comp
-L Interface_USB:CP2102N-A01-GQFN28 U9
+L Interface_USB:CP2102N-A01-GQFN28 U13
 U 1 1 62822250
 P 5200 3850
-F 0 "U9" H 4350 2800 50  0000 C CNN
+F 0 "U13" H 4350 2800 50  0000 C CNN
 F 1 "CP2102N-A01-GQFN28" H 4300 2700 50  0000 C CNN
 F 2 "Package_DFN_QFN:QFN-28-1EP_5x5mm_P0.5mm_EP3.35x3.35mm" H 5650 2650 50  0001 L CNN
@@
 DATA-
 $Comp
-L Device:R R20
+L Device:R R37
 U 1 1 62827308
 P 4600 2800
-F 0 "R20" H 4400 2850 50  0000 L CNN
+F 0 "R37" H 4400 2850 50  0000 L CNN
 F 1 "1k" H 4450 2750 50  0000 L CNN
 F 2 "Resistor_SMD:R_0603_1608Metric" V 4530 2800 50  0001 C CNN
@@
 	4700 2950 4600 2950
 $Comp
-L power:GND #PWR0262
+L power:GND #PWR0220
 U 1 1 6282ED0D
 P 5200 5150
-F 0 "#PWR0262" H 5200 4900 50  0001 C CNN
+F 0 "#PWR0220" H 5200 4900 50  0001 C CNN
 F 1 "GND" H 5205 4977 50  0000 C CNN
 F 2 "" H 5200 5150 50  0001 C CNN
@@
 	5200 2100 5200 2250
 $Comp
-L Personal_Misc:+3V3_USB #PWR0263
+L Personal_Misc:+3V3_USB #PWR0216
 U 1 1 6283201D
 P 4600 2650
-F 0 "#PWR0263" H 4600 2500 50  0001 C CNN
+F 0 "#PWR0216" H 4600 2500 50  0001 C CNN
 F 1 "+3V3_USB" H 4350 2750 50  0000 C CNN
 F 2 "" H 4600 2650 50  0001 C CNN
@@
 $EndComp
 $Comp
-L Device:C C83
+L Device:C C112
 U 1 1 62832576
 P 5350 2250
-F 0 "C83" V 5400 2350 50  0000 C CNN
+F 0 "C112" V 5400 2350 50  0000 C CNN
 F 1 "4.7u" V 5300 2400 50  0000 C CNN
 F 2 "Capacitor_SMD:C_0603_1608Metric" H 5388 2100 50  0001 C CNN
@@
 	5200 2250 5200 2450
 $Comp
-L Device:C C85
+L Device:C C114
 U 1 1 62832EDD
 P 5350 2450
-F 0 "C85" V 5300 2550 50  0000 C CNN
+F 0 "C114" V 5300 2550 50  0000 C CNN
 F 1 "100n" V 5400 2600 50  0000 C CNN
 F 2 "Capacitor_SMD:C_0603_1608Metric" H 5388 2300 50  0001 C CNN
@@
 	5200 2450 5200 2550
 $Comp
-L Device:C C82
+L Device:C C111
 U 1 1 62833498
 P 4950 2250
-F 0 "C82" V 5000 2100 50  0000 C CNN
+F 0 "C111" V 5000 2100 50  0000 C CNN
 F 1 "4.7u" V 4900 2100 50  0000 C CNN
 F 2 "Capacitor_SMD:C_0603_1608Metric" H 4988 2100 50  0001 C CNN
@@
 	5100 2250 5100 2450
 $Comp
-L Device:C C84
+L Device:C C113
 U 1 1 62833799
 P 4950 2450
-F 0 "C84" V 4900 2300 50  0000 C CNN
+F 0 "C113" V 4900 2300 50  0000 C CNN
 F 1 "100n" V 5000 2300 50  0000 C CNN
 F 2 "Capacitor_SMD:C_0603_1608Metric" H 4988 2300 50  0001 C CNN
@@
 	5100 2450 5100 2550
 $Comp
-L power:GND #PWR0264
+L power:GND #PWR0215
 U 1 1 62833E21
 P 5550 2350
-F 0 "#PWR0264" H 5550 2100 50  0001 C CNN
+F 0 "#PWR0215" H 5550 2100 50  0001 C CNN
 F 1 "GND" V 5555 2222 50  0000 R CNN
 F 2 "" H 5550 2350 50  0001 C CNN
@@
 Connection ~ 5550 2350
 $Comp
-L power:GND #PWR0265
+L power:GND #PWR0214
 U 1 1 628344DA
 P 4750 2350
-F 0 "#PWR0265" H 4750 2100 50  0001 C CNN
+F 0 "#PWR0214" H 4750 2100 50  0001 C CNN
 F 1 "GND" V 4755 2222 50  0000 R CNN
 F 2 "" H 4750 2350 50  0001 C CNN
@@
 RX
 $Comp
-L Personal_Misc:+3V3_USB #PWR0267
+L Personal_Misc:+3V3_USB #PWR0213
 U 1 1 62830F6B
 P 5200 2100
-F 0 "#PWR0267" H 5200 1950 50  0001 C CNN
+F 0 "#PWR0213" H 5200 1950 50  0001 C CNN
 F 1 "+3V3_USB" H 5350 2250 50  0000 C CNN
 F 2 "" H 5200 2100 50  0001 C CNN
@@
 $EndComp
 $Comp
-L Personal_Misc:+3V3_USB #PWR0268
+L Personal_Misc:+3V3_USB #PWR0219
 U 1 1 62846A4C
 P 7350 4400
-F 0 "#PWR0268" H 7350 4250 50  0001 C CNN
+F 0 "#PWR0219" H 7350 4250 50  0001 C CNN
 F 1 "+3V3_USB" V 7350 4700 50  0000 C CNN
 F 2 "" H 7350 4400 50  0001 C CNN
@@
 $EndComp
 $Comp
-L Device:R R23
+L Device:R R40
 U 1 1 62847DBA
 P 7050 4350
-F 0 "R23" V 6950 4350 50  0000 C CNN
+F 0 "R40" V 6950 4350 50  0000 C CNN
 F 1 "180" V 7050 4350 50  0000 C CNN
 F 2 "Resistor_SMD:R_0603_1608Metric" V 6980 4350 50  0001 C CNN
@@
 $EndComp
 $Comp
-L Device:R R24
+L Device:R R41
 U 1 1 6284804E
 P 7050 4450
-F 0 "R24" V 7150 4450 50  0000 C CNN
+F 0 "R41" V 7150 4450 50  0000 C CNN
 F 1 "180" V 7050 4450 50  0000 C CNN
 F 2 "Resistor_SMD:R_0603_1608Metric" V 6980 4450 50  0001 C CNN
@@
 NoConn ~ 5700 3450
 $Comp
-L Device:R R22
+L Device:R R39
 U 1 1 6285B100
 P 6050 3650
-F 0 "R22" V 5950 3650 50  0000 C CNN
+F 0 "R39" V 5950 3650 50  0000 C CNN
 F 1 "180" V 6050 3650 50  0000 C CNN
 F 2 "Resistor_SMD:R_0603_1608Metric" V 5980 3650 50  0001 C CNN
@@
 $EndComp
 $Comp
-L power:GND #PWR0269
+L power:GND #PWR0218
 U 1 1 6285D5A3
 P 7100 3650
-F 0 "#PWR0269" H 7100 3400 50  0001 C CNN
+F 0 "#PWR0218" H 7100 3400 50  0001 C CNN
 F 1 "GND" V 7105 3522 50  0000 R CNN
 F 2 "" H 7100 3650 50  0001 C CNN
@@
 	5700 3650 5800 3650
 $Comp
-L Device:R R21
+L Device:R R38
 U 1 1 6285E54F
 P 6050 3550
-F 0 "R21" V 6150 3550 50  0000 C CNN
+F 0 "R38" V 6150 3550 50  0000 C CNN
 F 1 "10k" V 6050 3550 50  0000 C CNN
 F 2 "Resistor_SMD:R_0603_1608Metric" V 5980 3550 50  0001 C CNN
@@
 	3800 1850 3800 5400
 $Comp
-L Personal_Misc:+5V_USB #PWR0277
+L Personal_Misc:+5V_USB #PWR0212
 U 1 1 62789052
 P 5100 2100
-F 0 "#PWR0277" H 5100 1950 50  0001 C CNN
+F 0 "#PWR0212" H 5100 1950 50  0001 C CNN
 F 1 "+5V_USB" H 4950 2250 50  0000 C CNN
 F 2 "" H 5100 2100 50  0001 C CNN
@@
 $EndComp
 $Comp
-L Personal_Misc:+5V_USB #PWR0278
+L Personal_Misc:+5V_USB #PWR0217
 U 1 1 6278A4CB
 P 4600 3150
-F 0 "#PWR0278" H 4600 3000 50  0001 C CNN
+F 0 "#PWR0217" H 4600 3000 50  0001 C CNN
 F 1 "+5V_USB" H 4400 3250 50  0000 C CNN
 F 2 "" H 4600 3150 50  0001 C CNN
