File: PCBV1/Processor.sch (KiCad schematic (older format))
At the start: 41 parts, among them U8 MCIMX6Y2CVM08AB

Commit message: Laid final hands on Wi-Fi and all circuits. Started work on PCB.
Parts:
- added C70, C72, C74, C77: 24p, Capacitor_SMD:C_0402_1005Metric, symbol Device:C
- added R33, R34: 4.7k, Resistor_SMD:R_0603_1608Metric, symbol Device:R
- added R35: 2.2M, Resistor_SMD:R_0603_1608Metric, symbol Device:R
- added SW2: SW_DIP_x02, Button_Switch_SMD:SW_DIP_SPSTx02_Slide_6.7x6.64mm_W6.73mm_P2.54mm_LowProfile_JPin, symbol Switch:SW_DIP_x02
- added Y2: ECS.32712.512, Personal_Actives:ECS32712512TR, symbol Device:Crystal
- added Y3: ECS2401823BJTM, Personal_Actives:ECS2401823BJTMTR, symbol Device:Crystal_GND24_Small
- C100: renamed from C71; footprint Capacitor_SMD:C_0603_1608Metric -> Capacitor_SMD:C_0402_1005Metric
- C101: renamed from C72; footprint Capacitor_SMD:C_0603_1608Metric -> Capacitor_SMD:C_0402_1005Metric
- C102: renamed from C73; footprint Capacitor_SMD:C_0603_1608Metric -> Capacitor_SMD:C_0402_1005Metric
- C103: renamed from C74; footprint Capacitor_SMD:C_0603_1608Metric -> Capacitor_SMD:C_0402_1005Metric
- C106: renamed from C77; footprint Capacitor_SMD:C_0603_1608Metric -> Capacitor_SMD:C_0402_1005Metric
- C107: renamed from C78; footprint Capacitor_SMD:C_0603_1608Metric -> Capacitor_SMD:C_0402_1005Metric
- C108: renamed from C79; footprint Capacitor_SMD:C_0603_1608Metric -> Capacitor_SMD:C_0402_1005Metric
- C109: renamed from C80; footprint Capacitor_SMD:C_0603_1608Metric -> Capacitor_SMD:C_0402_1005Metric
- C110: renamed from C81; footprint Capacitor_SMD:C_0603_1608Metric -> Capacitor_SMD:C_0402_1005Metric
- C68: renamed from C43; footprint Capacitor_SMD:C_0603_1608Metric -> Capacitor_SMD:C_0402_1005Metric
- C69: renamed from C44; footprint Capacitor_SMD:C_0603_1608Metric -> Capacitor_SMD:C_0402_1005Metric
- C71: renamed from C45; footprint Capacitor_SMD:C_0603_1608Metric -> Capacitor_SMD:C_0402_1005Metric
- C73: renamed from C46; footprint Capacitor_SMD:C_0603_1608Metric -> Capacitor_SMD:C_0402_1005Metric
- C75: renamed from C47; footprint Capacitor_SMD:C_0603_1608Metric -> Capacitor_SMD:C_0402_1005Metric
- C76: renamed from C48; footprint Capacitor_SMD:C_0603_1608Metric -> Capacitor_SMD:C_0402_1005Metric
- C78: renamed from C49; footprint Capacitor_SMD:C_0603_1608Metric -> Capacitor_SMD:C_0402_1005Metric
- C79: renamed from C50; footprint Capacitor_SMD:C_0603_1608Metric -> Capacitor_SMD:C_0402_1005Metric
- C81: renamed from C52; footprint Capacitor_SMD:C_0603_1608Metric -> Capacitor_SMD:C_0402_1005Metric
- C82: renamed from C53; footprint Capacitor_SMD:C_0603_1608Metric -> Capacitor_SMD:C_0402_1005Metric
- C84: renamed from C55; footprint Capacitor_SMD:C_0603_1608Metric -> Capacitor_SMD:C_0402_1005Metric
- C85: renamed from C56; footprint Capacitor_SMD:C_0603_1608Metric -> Capacitor_SMD:C_0402_1005Metric
- C86: renamed from C57; footprint Capacitor_SMD:C_0603_1608Metric -> Capacitor_SMD:C_0402_1005Metric
- C88: renamed from C59; footprint Capacitor_SMD:C_0603_1608Metric -> Capacitor_SMD:C_0402_1005Metric
- C89: renamed from C60; footprint Capacitor_SMD:C_0603_1608Metric -> Capacitor_SMD:C_0402_1005Metric
- C90: renamed from C61; footprint Capacitor_SMD:C_0603_1608Metric -> Capacitor_SMD:C_0402_1005Metric
- C91: renamed from C62; footprint Capacitor_SMD:C_0603_1608Metric -> Capacitor_SMD:C_0402_1005Metric
- C93: renamed from C64; footprint Capacitor_SMD:C_0603_1608Metric -> Capacitor_SMD:C_0402_1005Metric
- C94: renamed from C65; footprint Capacitor_SMD:C_0603_1608Metric -> Capacitor_SMD:C_0402_1005Metric
- C95: renamed from C66; footprint Capacitor_SMD:C_0603_1608Metric -> Capacitor_SMD:C_0402_1005Metric
- C97: renamed from C68; footprint Capacitor_SMD:C_0603_1608Metric -> Capacitor_SMD:C_0402_1005Metric
- C98: renamed from C69; footprint Capacitor_SMD:C_0603_1608Metric -> Capacitor_SMD:C_0402_1005Metric
- renumbered C75 to C104, C76 to C105, C51 to C80, C54 to C83, C58 to C87, C63 to C92, C67 to C96, C70 to C99, R19 to R36, U8 to U1
Connections:
- net +3V3: now also R33.2, R34.2
- net GND: now also U1.M12 (NGND_KEL0), U1.N7 (TEST_MODE), C70.2, C72.2, C74.2, C77.2, R35.2, Y3.2, Y3.4
- net SD2_D3: now reaches U1.E1 (CSI_DATA03)
- net SD2_D2: now reaches U1.E2 (CSI_DATA02)
- net SD2_D1: now reaches U1.E3 (CSI_DATA01)
- net SD2_D0: now reaches U1.E4 (CSI_DATA00)
- net SD2_CLK: now reaches U1.F2 (CSI_VSYNC)
- net SD2_CMD: now reaches U1.F3 (CSI_HSYNC)
- net BM0: now reaches U1.T10 (BOOT_MODE0)
- net BM0: now also SW2.3
- net at U1.T11 (RTC_XTALI): now also C72.1, Y2.2
- net at U1.T16 (XTALI): now also C77.1, R35.1, Y3.3
- net at U1.T17 (XTALO): now also C74.1, Y3.1
- net BM1: now reaches U1.U10 (BOOT_MODE1)
- net BM1: now also SW2.4
- net at U1.U11 (RTC_XTALO): now also C70.1, Y2.1
- net SD_CLK renamed SD1_CLK
- net SD_CMD renamed SD1_CMD
- net SD_D0 renamed SD1_D0
- net SD_D1 renamed SD1_D1
- net SD_D2 renamed SD1_D2
- net SD_D3 renamed SD1_D3
- net ~SD_CD renamed ~SD1_CD
- new net: R34.1, SW2.2
- new net: R33.1, SW2.1
- no-connect marks 61 -> 83
Other:
- note added: "00: Boot from fuses\n01: Serial downloader\n10: Internal boot\n11: Reserver"
- note added: "Boot mode switches"
- note added: "Place resistor close to XTALI"
- note removed: "CONNECT CRYSTAL\nBIAS WITH RESISTOR"
- note removed: "CONNECT RTC CRYSTAL"
- note removed: "Overvej om LCD_DATA06 skal trækkes høj med pull-up"
