File: PCBV1/DDR.sch (KiCad schematic (older format))
At the start: 0 parts

Commit message: Added schematic for power through barrel jack and voltage converters, connected DRAM.
Parts:
- added C? (x15): 100 nF, symbol Device:C
- added C?: 22 µF, symbol Device:C
- added C?: 4.7 µF, symbol Device:C
- added R?: 240R, symbol Device:R
- added R? (x2): 1.5k, symbol Device:R
- added U?: MT41K128M16JT-125_K, Personal_ICs:MT41K128M16JT-125, symbol Personal_ICs:MT41K128M16JT-125_K
Connections:
- new net: R?.2, U?.L8 (ZQ)
- new net: C?.1, C?.2
- new net +1V35: C?.1, C?.1, C?.1, C?.1, C?.1, C?.1, C?.1, C?.1, C?.1, C?.1, C?.1, C?.1, C?.1, C?.1, R?.1, U?.A1 (VDDQ_1), U?.A8 (VDDQ_2), U?.B2 (VDD_1), U?.C1 (VDDQ_3), U?.C9 (VDDQ_4), U?.D2 (VDDQ_5), U?.D9 (VDD_2), U?.E9 (VDDQ_6), U?.F1 (VDDQ_7), U?.G7 (VDD_3), U?.H2 (VDDQ_8), U?.H9 (VDDQ_9), U?.K2 (VDD_4), U?.K8 (VDD_5), U?.N1 (VDD_6), U?.N9 (VDD_7), U?.R1 (VDD_8), U?.R9 (VDD_9)
- new net DDR_A0: U?.N3 (A0)
- new net DDR_A1: U?.P7 (A1)
- new net DDR_A10: U?.L7 (A10/AP)
- new net DDR_A11: U?.R7 (A11)
- new net DDR_A12: U?.N7 (A12/BC#)
- new net DDR_A13: U?.T3 (A13)
- new net DDR_A2: U?.P3 (A2)
- new net DDR_A3: U?.N2 (A3)
- new net DDR_A4: U?.P8 (A4)
- new net DDR_A5: U?.P2 (A5)
- new net DDR_A6: U?.R8 (A6)
- new net DDR_A7: U?.R2 (A7)
- new net DDR_A8: U?.T8 (A8)
- new net DDR_A9: U?.R3 (A9)
- new net DDR_BA0: U?.M2 (BA0)
- new net DDR_BA1: U?.N8 (BA1)
- new net DDR_BA2: U?.M3 (BA2)
- new net DDR_CK: U?.J7 (CK)
- new net DDR_CKE: U?.K9 (CKE)
- new net DDR_D0: U?.E3 (DQ0)
- new net DDR_D1: U?.F7 (DQ1)
- new net DDR_D10: U?.C8 (DQ10)
- new net DDR_D11: U?.C2 (DQ11)
- new net DDR_D12: U?.A7 (DQ12)
- new net DDR_D13: U?.A2 (DQ13)
- new net DDR_D14: U?.B8 (DQ14)
- new net DDR_D15: U?.A3 (DQ15)
- new net DDR_D2: U?.F2 (DQ2)
- new net DDR_D3: U?.F8 (DQ3)
- new net DDR_D4: U?.H3 (DQ4)
- new net DDR_D5: U?.H8 (DQ5)
- new net DDR_D6: U?.G2 (DQ6)
- new net DDR_D7: U?.H7 (DQ7)
- new net DDR_D8: U?.D7 (DQ8)
- new net DDR_D9: U?.C3 (DQ9)
- new net DDR_LDM: U?.E7 (LDM)
- new net DDR_LDQS: U?.F3 (LDQS)
- new net DDR_ODT: U?.K1 (ODT)
- new net DDR_RST: U?.T2 (RESET#)
- new net DDR_UDM: U?.D3 (UDM)
- new net DDR_UDQS: U?.C7 (UDQS)
- new net DRAM_VREF: C?.1, C?.2, R?.1, R?.2, U?.H1 (VREFDQ), U?.M8 (VREFCA)
- new net GND: C?.1, C?.2, C?.2, C?.2, C?.2, C?.2, C?.2, C?.2, C?.2, C?.2, C?.2, C?.2, C?.2, C?.2, C?.2, C?.2, R?.1, R?.2, U?.A9 (VSS_1), U?.B1 (VSSQ_1), U?.B3 (VSS_2), U?.B9 (VSSQ_2), U?.D1 (VSSQ_3), U?.D8 (VSSQ_4), U?.E1 (VSS_3), U?.E2 (VSSQ_5), U?.E8 (VSSQ_6), U?.F9 (VSSQ_7), U?.G1 (VSSQ_8), U?.G8 (VSS_4), U?.G9 (VSSQ_9), U?.J2 (VSS_5), U?.J8 (VSS_6), U?.M1 (VSS_7), U?.M9 (VSS_8), U?.P1 (VSS_9), U?.P9 (VSS_10), U?.T1 (VSS_11), U?.T9 (VSS_12)
- new net ~DDR_CAS: U?.K3 (CAS#)
- new net ~DDR_CK: U?.K7 (CK#)
- new net ~DDR_CS: U?.L2 (CS#)
- new net ~DDR_LDQS: U?.G3 (LDQS#)
- new net ~DDR_RAS: U?.J3 (RAS#)
- new net ~DDR_UDQS: U?.B7 (UDQS#)
- new net ~DDR_WE: U?.L3 (WE#)
- no-connect marks 0 -> 6
Other:
- note added: "2 Gb (128 x 16) DDR3L"
- note added: "Clock termination?"
- note added: "Decoupling"
- note added: "Reference voltage generation"
- note added: "Resistors must be 1% or better tolerance."

Commit message: Changes to DDR schematic.
Parts:
- added R? (x2): 10k, symbol Device:R
- added R?: 470R, symbol Device:R
Connections:
- net DDR_CK: now also R?.1
- net DDR_CKE: now also R?.2
- net DDR_RST: now also R?.2
- net GND: now also R?.1, R?.1
- net ~DDR_CK: now also R?.2
Other:
- note removed: "Clock termination?"
- moved on the sheet: R?
Changed lines of the file:
@@
 Wire Wire Line
 	3750 2100 3550 2100
-Wire Wire Line
-	3550 3600 3750 3600
 $Comp
 L Device:R R?
 U 1 1 602AEFA8
-P 3900 3600
-F 0 "R?" V 3900 3800 50  0000 C CNN
-F 1 "240R" V 3900 3600 50  0000 C CNN
-F 2 "" V 3830 3600 50  0001 C CNN
-F 3 "~" H 3900 3600 50  0001 C CNN
-	1    3900 3600
+P 4150 3600
+F 0 "R?" V 4150 3800 50  0000 C CNN
+F 1 "240R" V 4150 3600 50  0000 C CNN
+F 2 "" V 4080 3600 50  0001 C CNN
+F 3 "~" H 4150 3600 50  0001 C CNN
+	1    4150 3600
 	0    1    1    0
 $EndComp
 Wire Wire Line
-	4050 3600 4250 3600
+	4300 3600 4500 3600
 $Comp
 L power:GND #PWR?
 U 1 1 602AFE78
-P 4250 3600
-F 0 "#PWR?" H 4250 3350 50  0001 C CNN
-F 1 "GND" V 4255 3472 50  0000 R CNN
-F 2 "" H 4250 3600 50  0001 C CNN
-F 3 "" H 4250 3600 50  0001 C CNN
-	1    4250 3600
+P 4500 3600
+F 0 "#PWR?" H 4500 3350 50  0001 C CNN
+F 1 "GND" V 4505 3472 50  0000 R CNN
+F 2 "" H 4500 3600 50  0001 C CNN
+F 3 "" H 4500 3600 50  0001 C CNN
+	1    4500 3600
 	0    -1   -1   0
 $EndComp
@@
 Text HLabel 3600 2900 2    50   Input ~ 0
 ~DDR_CK
-Wire Wire Line
-	3600 2900 3550 2900
-Wire Wire Line
-	3550 3100 3600 3100
 Text HLabel 3600 2800 2    50   Input ~ 0
 ~DDR_CAS
@@
 Text HLabel 3600 2300 2    50   Input ~ 0
 DDR_CK
-Wire Wire Line
-	3600 2300 3550 2300
 Text HLabel 3600 2200 2    50   Input ~ 0
 ~DDR_RAS
@@
 Wire Wire Line
 	3750 6100 3550 6100
-Wire Wire Line
-	3550 6300 3600 6300
 Text HLabel 3600 6300 2    50   Input ~ 0
 DDR_RST
@@
 Text Notes 5200 3450 0    50   ~ 0
 Reference voltage generation
-Text Notes 6400 4900 0    100  ~ 0
-Clock termination?
+$Comp
+L Device:R R?
+U 1 1 602DD0F6
+P 4150 6300
+F 0 "R?" V 4150 6500 50  0000 C CNN
+F 1 "10k" V 4150 6300 50  0000 C CNN
+F 2 "" V 4080 6300 50  0001 C CNN
+F 3 "~" H 4150 6300 50  0001 C CNN
+	1    4150 6300
+	0    1    1    0
+$EndComp
+Wire Wire Line
+	4300 6300 4500 6300
+$Comp
+L power:GND #PWR?
+U 1 1 602DD0FD
+P 4500 6300
+F 0 "#PWR?" H 4500 6050 50  0001 C CNN
+F 1 "GND" V 4505 6172 50  0000 R CNN
+F 2 "" H 4500 6300 50  0001 C CNN
+F 3 "" H 4500 6300 50  0001 C CNN
+	1    4500 6300
+	0    -1   -1   0
+$EndComp
+Wire Wire Line
+	3550 6300 4000 6300
+$Comp
+L Device:R R?
+U 1 1 602E7798
+P 4150 3100
+F 0 "R?" V 4150 3300 50  0000 C CNN
+F 1 "10k" V 4150 3100 50  0000 C CNN
+F 2 "" V 4080 3100 50  0001 C CNN
+F 3 "~" H 4150 3100 50  0001 C CNN
+	1    4150 3100
+	0    1    1    0
+$EndComp
+Wire Wire Line
+	4300 3100 4500 3100
+$Comp
+L power:GND #PWR?
+U 1 1 602E779F
+P 4500 3100
+F 0 "#PWR?" H 4500 2850 50  0001 C CNN
+F 1 "GND" V 4505 2972 50  0000 R CNN
+F 2 "" H 4500 3100 50  0001 C CNN
+F 3 "" H 4500 3100 50  0001 C CNN
+	1    4500 3100
+	0    -1   -1   0
+$EndComp
+Wire Wire Line
+	3550 3100 4000 3100
+Wire Wire Line
+	3550 3600 4000 3600
+Wire Wire Line
+	3550 2300 4350 2300
+Wire Wire Line
+	3550 2900 4350 2900
+$Comp
+L Device:R R?
+U 1 1 60314802
+P 4350 2600
+F 0 "R?" H 4420 2646 50  0000 L CNN
+F 1 "470R" H 4420 2555 50  0000 L CNN
+F 2 "" V 4280 2600 50  0001 C CNN
+F 3 "~" H 4350 2600 50  0001 C CNN
+	1    4350 2600
+	1    0    0    -1
+$EndComp
+Wire Wire Line
+	4350 2450 4350 2300
+Wire Wire Line
+	4350 2750 4350 2900
 $EndSCHEMATC

Commit message: Many minor changes to component footprints and schematics.
Parts:
- C26, C27, C28, C29, C30, C31, C32, C33, C34, C35, C36, C38, C40, C41, C42: renamed from C?; value 100 nF -> 100n; footprint (none) -> Capacitor_SMD:C_0603_1608Metric
- C37: renamed from C?; value 22 µF -> 100n; footprint (none) -> Capacitor_SMD:C_0603_1608Metric
- C39: renamed from C?; value 4.7 µF -> 4.7µ; footprint (none) -> Capacitor_SMD:C_0603_1608Metric
- R13, R14, R15, R16, R17, R18: renamed from R?; footprint (none) -> Resistor_SMD:R_0603_1608Metric
- gave numbers to parts that had none: 1

Commit message: Laid final hands on Wi-Fi and all circuits. Started work on PCB.
Parts:
- renumbered C26 to C51, C27 to C52, C28 to C53, C29 to C54, C30 to C55, C31 to C56, C32 to C57, C33 to C58, C34 to C59, C35 to C60, C36 to C61, C37 to C62, C38 to C63, C39 to C64, C40 to C65, C41 to C66, C42 to C67, R13 to R27, R14 to R28, R15 to R29, R16 to R30, R17 to R31, R18 to R32, U7 to U2
