File: PCBV1/Video.sch (KiCad schematic (older format))
At the start: 21 parts, among them U3 TFP410PAP

Commit message: Laid final hands on Wi-Fi and all circuits. Started work on PCB.
Parts:
- renumbered C3 to C19, C4 to C20, C5 to C21, C6 to C22, C7 to C23, C8 to C24, C9 to C25, C10 to C26, C11 to C27, C12 to C28, C13 to C29, FB1 to FB3, FB2 to FB4, FB3 to FB5, R2 to R14, R3 to R15, R4 to R16, R5 to R17, R6 to R18, R7 to R19, U3 to U7
Changed lines of the file:
@@
 Sheet 3 8
 Title "Smart Mirror"
-Date "2022-04-22"
+Date "2022-05-11"
 Rev "1.0"
 Comp "University of Southern Denmark"
@@
 $EndDescr
 $Comp
-L Video:TFP410PAP U3
+L Video:TFP410PAP U7
 U 1 1 61CD7FE8
 P 4500 3450
-F 0 "U3" H 5350 1350 50  0000 C CNN
+F 0 "U7" H 5350 1350 50  0000 C CNN
 F 1 "TFP410PAP" H 5350 1200 50  0000 C CNN
 F 2 "Package_QFP:HTQFP-64-1EP_10x10mm_P0.5mm_EP8x8mm_Mask4.4x4.4mm_ThermalVias" H 4550 1050 50  0001 C CNN
@@
 	5400 2950 5200 2950
 $Comp
-L power:GND #PWR0111
+L power:GND #PWR037
 U 1 1 61CE0BED
 P 4450 900
-F 0 "#PWR0111" H 4450 650 50  0001 C CNN
+F 0 "#PWR037" H 4450 650 50  0001 C CNN
 F 1 "GND" H 4455 727 50  0000 C CNN
 F 2 "" H 4450 900 50  0001 C CNN
@@
 	5350 2750 5200 2750
 $Comp
-L power:GND #PWR0112
+L power:GND #PWR043
 U 1 1 62640B01
 P 5200 5550
-F 0 "#PWR0112" H 5200 5300 50  0001 C CNN
+F 0 "#PWR043" H 5200 5300 50  0001 C CNN
 F 1 "GND" V 5200 5350 50  0000 C CNN
 F 2 "" H 5200 5550 50  0001 C CNN
@@
 CLK
 $Comp
-L Device:R R7
+L Device:R R19
 U 1 1 6268C968
 P 3550 5550
-F 0 "R7" V 3450 5550 50  0000 C CNN
+F 0 "R19" V 3450 5550 50  0000 C CNN
 F 1 "4.7k" V 3550 5550 50  0000 C CNN
 F 2 "Resistor_SMD:R_0603_1608Metric" V 3480 5550 50  0001 C CNN
@@
 $EndComp
 $Comp
-L power:+3V3 #PWR0113
+L power:+3V3 #PWR042
 U 1 1 6268DBB5
 P 3300 5550
-F 0 "#PWR0113" H 3300 5400 50  0001 C CNN
+F 0 "#PWR042" H 3300 5400 50  0001 C CNN
 F 1 "+3V3" V 3300 5750 50  0000 C CNN
 F 2 "" H 3300 5550 50  0001 C CNN
@@
 	4000 6300 3900 6300
 $Comp
-L power:GND #PWR0114
+L power:GND #PWR045
 U 1 1 6268433D
 P 3850 6300
-F 0 "#PWR0114" H 3850 6050 50  0001 C CNN
+F 0 "#PWR045" H 3850 6050 50  0001 C CNN
 F 1 "GND" V 3850 6100 50  0000 C CNN
 F 2 "" H 3850 6300 50  0001 C CNN
@@
 	5200 6600 5300 6600
 $Comp
-L power:GND #PWR0115
+L power:GND #PWR046
 U 1 1 6267D9D2
 P 5300 6600
-F 0 "#PWR0115" H 5300 6350 50  0001 C CNN
+F 0 "#PWR046" H 5300 6350 50  0001 C CNN
 F 1 "GND" V 5300 6400 50  0000 C CNN
 F 2 "" H 5300 6600 50  0001 C CNN
@@
 	5000 6000 5200 6000
 $Comp
-L power:GND #PWR0116
+L power:GND #PWR044
 U 1 1 6267793B
 P 5300 6000
-F 0 "#PWR0116" H 5300 5750 50  0001 C CNN
+F 0 "#PWR044" H 5300 5750 50  0001 C CNN
 F 1 "GND" V 5300 5800 50  0000 C CNN
 F 2 "" H 5300 6000 50  0001 C CNN
@@
 	4600 5850 4900 5850
 $Comp
-L Device:C C5
+L Device:C C21
 U 1 1 6265B774
 P 4850 6000
-F 0 "C5" V 4900 6050 50  0000 L CNN
+F 0 "C21" V 4900 6050 50  0000 L CNN
 F 1 "10n" V 4800 6050 50  0000 L CNN
 F 2 "Capacitor_SMD:C_0603_1608Metric" H 4888 5850 50  0001 C CNN
@@
 $EndComp
 $Comp
-L Device:C C6
+L Device:C C22
 U 1 1 6265B335
 P 5050 6150
-F 0 "C6" V 5100 6200 50  0000 L CNN
+F 0 "C22" V 5100 6200 50  0000 L CNN
 F 1 "10n" V 5000 6200 50  0000 L CNN
 F 2 "Capacitor_SMD:C_0603_1608Metric" H 5088 6000 50  0001 C CNN
@@
 $EndComp
 $Comp
-L Device:C C9
+L Device:C C25
 U 1 1 62656CDC
 P 5050 6450
-F 0 "C9" V 5100 6500 50  0000 L CNN
+F 0 "C25" V 5100 6500 50  0000 L CNN
 F 1 "10n" V 5000 6500 50  0000 L CNN
 F 2 "Capacitor_SMD:C_0603_1608Metric" H 5088 6300 50  0001 C CNN
@@
 	4500 7450 4500 7400
 $Comp
-L Device:Ferrite_Bead_Small FB3
+L Device:Ferrite_Bead_Small FB5
 U 1 1 62635C99
 P 4500 7300
-F 0 "FB3" H 4600 7300 50  0000 L CNN
+F 0 "FB5" H 4600 7300 50  0000 L CNN
 F 1 "600R" H 4600 7200 50  0000 L CNN
 F 2 "Inductor_SMD:L_0603_1608Metric" V 4430 7300 50  0001 C CNN
@@
 $EndComp
 $Comp
-L Device:Ferrite_Bead_Small FB1
+L Device:Ferrite_Bead_Small FB3
 U 1 1 62635733
 P 4400 7150
-F 0 "FB1" H 4200 7200 50  0000 L CNN
+F 0 "FB3" H 4200 7200 50  0000 L CNN
 F 1 "600R" H 4150 7100 50  0000 L CNN
 F 2 "Inductor_SMD:L_0603_1608Metric" V 4330 7150 50  0001 C CNN
@@
 $EndComp
 $Comp
-L Device:Ferrite_Bead_Small FB2
+L Device:Ferrite_Bead_Small FB4
 U 1 1 6263496D
 P 4600 7150
-F 0 "FB2" H 4700 7196 50  0000 L CNN
+F 0 "FB4" H 4700 7196 50  0000 L CNN
 F 1 "600R" H 4700 7105 50  0000 L CNN
 F 2 "Inductor_SMD:L_0603_1608Metric" V 4530 7150 50  0001 C CNN
@@
 	4300 5850 4600 5850
 $Comp
-L Device:C C10
+L Device:C C26
 U 1 1 62623544
 P 4150 6600
-F 0 "C10" V 4100 6450 50  0000 L CNN
+F 0 "C26" V 4100 6450 50  0000 L CNN
 F 1 "22µ" V 4200 6400 50  0000 L CNN
 F 2 "Capacitor_SMD:C_0603_1608Metric" H 4188 6450 50  0001 C CNN
@@
 $EndComp
 $Comp
-L Device:C C7
+L Device:C C23
 U 1 1 626231AD
 P 4150 6300
-F 0 "C7" V 4100 6150 50  0000 L CNN
+F 0 "C23" V 4100 6150 50  0000 L CNN
 F 1 "22µ" V 4200 6100 50  0000 L CNN
 F 2 "Capacitor_SMD:C_0603_1608Metric" H 4188 6150 50  0001 C CNN
@@
 $EndComp
 $Comp
-L Device:C C11
+L Device:C C27
 U 1 1 6261D1F6
 P 4850 6600
-F 0 "C11" V 4900 6650 50  0000 L CNN
+F 0 "C27" V 4900 6650 50  0000 L CNN
 F 1 "10n" V 4800 6650 50  0000 L CNN
 F 2 "Capacitor_SMD:C_0603_1608Metric" H 4888 6450 50  0001 C CNN
@@
 $EndComp
 $Comp
-L Device:C C8
+L Device:C C24
 U 1 1 61D029E9
 P 4850 6300
-F 0 "C8" V 4900 6350 50  0000 L CNN
+F 0 "C24" V 4900 6350 50  0000 L CNN
 F 1 "10n" V 4800 6350 50  0000 L CNN
 F 2 "Capacitor_SMD:C_0603_1608Metric" H 4888 6150 50  0001 C CNN
@@
 $EndComp
 $Comp
-L Device:C C4
+L Device:C C20
 U 1 1 61D0235B
 P 5050 5850
-F 0 "C4" V 5100 5900 50  0000 L CNN
+F 0 "C20" V 5100 5900 50  0000 L CNN
 F 1 "10n" V 5000 5900 50  0000 L CNN
 F 2 "Capacitor_SMD:C_0603_1608Metric" H 5088 5700 50  0001 C CNN
@@
 $EndComp
 $Comp
-L Device:C C3
+L Device:C C19
 U 1 1 61D0075D
 P 4150 5850
-F 0 "C3" V 4100 5700 50  0000 L CNN
+F 0 "C19" V 4100 5700 50  0000 L CNN
 F 1 "22µ" V 4200 5650 50  0000 L CNN
 F 2 "Capacitor_SMD:C_0603_1608Metric" H 4188 5700 50  0001 C CNN
@@
 $EndComp
 $Comp
-L power:+3V3 #PWR0117
+L power:+3V3 #PWR047
 U 1 1 61CF8EDB
 P 4500 7450
-F 0 "#PWR0117" H 4500 7300 50  0001 C CNN
+F 0 "#PWR047" H 4500 7300 50  0001 C CNN
 F 1 "+3V3" H 4515 7623 50  0000 C CNN
 F 2 "" H 4500 7450 50  0001 C CNN
@@
 $EndComp
 $Comp
-L Device:C C12
+L Device:C C28
 U 1 1 626D2609
 P 5050 6750
-F 0 "C12" V 5100 6800 50  0000 L CNN
+F 0 "C28" V 5100 6800 50  0000 L CNN
 F 1 "10n" V 5000 6800 50  0000 L CNN
 F 2 "Capacitor_SMD:C_0603_1608Metric" H 5088 6600 50  0001 C CNN
@@
 $EndComp
 $Comp
-L Device:C C13
+L Device:C C29
 U 1 1 626D2B70
 P 4850 6900
-F 0 "C13" V 4900 6950 50  0000 L CNN
+F 0 "C29" V 4900 6950 50  0000 L CNN
 F 1 "10n" V 4800 6950 50  0000 L CNN
 F 2 "Capacitor_SMD:C_0603_1608Metric" H 4888 6750 50  0001 C CNN
@@
 Connection ~ 5200 6750
 $Comp
-L Device:R R6
+L Device:R R18
 U 1 1 626F776B
 P 3550 5350
-F 0 "R6" V 3450 5350 50  0000 C CNN
+F 0 "R18" V 3450 5350 50  0000 C CNN
 F 1 "510" V 3550 5350 50  0000 C CNN
 F 2 "Resistor_SMD:R_0603_1608Metric" V 3480 5350 50  0001 C CNN
@@
 	5200 2250 5300 2250
 $Comp
-L Device:R R4
+L Device:R R16
 U 1 1 627033B6
 P 5450 2250
-F 0 "R4" V 5350 2250 50  0000 C CNN
+F 0 "R16" V 5350 2250 50  0000 C CNN
 F 1 "4.7k" V 5450 2250 50  0000 C CNN
 F 2 "Resistor_SMD:R_0603_1608Metric" V 5380 2250 50  0001 C CNN
@@
 	5600 2250 5700 2250
 $Comp
-L power:GND #PWR0118
+L power:GND #PWR040
 U 1 1 6270C44E
 P 5700 2250
-F 0 "#PWR0118" H 5700 2000 50  0001 C CNN
+F 0 "#PWR040" H 5700 2000 50  0001 C CNN
 F 1 "GND" V 5700 2050 50  0000 C CNN
 F 2 "" H 5700 2250 50  0001 C CNN
@@
 	5200 2350 5300 2350
 $Comp
-L Device:R R5
+L Device:R R17
 U 1 1 6270E5B0
 P 5450 2350
-F 0 "R5" V 5550 2350 50  0000 C CNN
+F 0 "R17" V 5550 2350 50  0000 C CNN
 F 1 "4.7k" V 5450 2350 50  0000 C CNN
 F 2 "Resistor_SMD:R_0603_1608Metric" V 5380 2350 50  0001 C CNN
@@
 	5600 2350 5700 2350
 $Comp
-L power:+3V3 #PWR0119
+L power:+3V3 #PWR041
 U 1 1 62712590
 P 5700 2350
-F 0 "#PWR0119" H 5700 2200 50  0001 C CNN
+F 0 "#PWR041" H 5700 2200 50  0001 C CNN
 F 1 "+3V3" V 5700 2550 50  0000 C CNN
 F 2 "" H 5700 2350 50  0001 C CNN
@@
 NoConn ~ 5200 2050
 $Comp
-L Device:R R3
+L Device:R R15
 U 1 1 6271884F
 P 5450 1850
-F 0 "R3" V 5350 1850 50  0000 C CNN
+F 0 "R15" V 5350 1850 50  0000 C CNN
 F 1 "4.7k" V 5450 1850 50  0000 C CNN
 F 2 "Resistor_SMD:R_0603_1608Metric" V 5380 1850 50  0001 C CNN
@@
 	5600 1850 5700 1850
 $Comp
-L power:GND #PWR0120
+L power:GND #PWR039
 U 1 1 62718856
 P 5700 1850
-F 0 "#PWR0120" H 5700 1600 50  0001 C CNN
+F 0 "#PWR039" H 5700 1600 50  0001 C CNN
 F 1 "GND" V 5700 1650 50  0000 C CNN
 F 2 "" H 5700 1850 50  0001 C CNN
@@
 	5200 1350 5300 1350
 $Comp
-L Device:R R2
+L Device:R R14
 U 1 1 62720A08
 P 5450 1350
-F 0 "R2" V 5550 1350 50  0000 C CNN
+F 0 "R14" V 5550 1350 50  0000 C CNN
 F 1 "4.7k" V 5450 1350 50  0000 C CNN
 F 2 "Resistor_SMD:R_0603_1608Metric" V 5380 1350 50  0001 C CNN
@@
 	5600 1350 5700 1350
 $Comp
-L power:+3V3 #PWR0121
+L power:+3V3 #PWR038
 U 1 1 62720A0F
 P 5700 1350
-F 0 "#PWR0121" H 5700 1200 50  0001 C CNN
+F 0 "#PWR038" H 5700 1200 50  0001 C CNN
 F 1 "+3V3" V 5700 1550 50  0000 C CNN
 F 2 "" H 5700 1350 50  0001 C CNN
